File: design_files/ASD2412.brd (EAGLE design)
At the start: 22.5 x 22.5 mm, 29 parts, among them J2 DF12-32-DS

Commit message: Update format
Other:
- board size 22.5 x 22.5 mm -> 20 x 20 mm
- board text added: "TinyCircuits.com"
- board text removed: "Tiny-Circuits.com"
